File: _autosave-Phoenix_Bot_arduino_shield.kicad_pcb (KiCad board)
At the start: 2 copper layers, 135.9 x 64.8 mm, 46 parts, among them J1 Analog_signal_male, J10 Ground, J11 Ground, J12 Ground, J13 12V_terminal, J14 PWN(10-5), J15 On Board Supply, J16 1x8 Male, J17 1x8 Male, J18 PWM_(6-1), J19 Analog_Pin_1, J2 Encoder_signal, J20 1x8 Female, J21 1x8 Female, J22 Serial, J23 ICSP, J24 Analog_Pin_2, J25 Digital_Pins, J27 Solenoid_terminal, J28 Solendoid_middle_terminal, J29 bottom_solenoid_terminal, J3 Servo_signal, J4 Analog_signal_female, J5 Analog_signal_power, J6 Servo_Power, J7 Encoder_Power, J8 Analog_Power_female, J9 Ground, q1 solenoid_1, q2 solenoid_4, q3 solenoid_3, q4 solenoid_5, q5 solenoid_3, q6 solenoid_6

Commit message: Began board layout
Routing:
- net +12V: track 210.6 -> 75.3 mm
- net /Drain_1: track 26.3 -> 11.8 mm
- net /Drain_3: track 46.0 -> 36.6 mm
- net /Drain_2: track 55.1 -> 60.3 mm
- net /Drain_5: track 31.5 -> 29.5 mm
- net /Drain_4: track 23.7 -> 25.0 mm
Other:
- net class Default: clearance 0.006 -> 0.1524; trace_width 0.006 -> 0.1524; via_dia 0.027 -> 0.6858; via_drill 0.013 -> 0.3302
- net class Powertrace: clearance 0.006 -> 0.254; trace_width 0.0544 -> 1.38176; via_dia 0.027 -> 0.6858; via_drill 0.013 -> 0.3302
- rule trace_clearance: 0.006 -> 0.1524
- rule trace_min: 0.006 -> 0.1524
- rule via_min_drill: 0.013 -> 0.3302
- rule via_min_size: 0.027 -> 0.6858

Commit message: More progress on Board, mapped except solenoids
Parts:
- removed J10, J11: Ground, Pin_Headers:Pin_Header_Straight_1x06_Pitch2.54mm
- removed J12, J9: Ground, Pin_Headers:Pin_Header_Straight_1x08_Pitch2.54mm
- removed J5: Analog_signal_power, Pin_Headers:Pin_Header_Straight_1x08_Pitch2.54mm
- J2: value Encoder_signal -> Encoder_Signal; footprint Pin_Headers:Pin_Header_Straight_1x06_Pitch2.54mm -> Pin_Headers:Pin_Header_Straight_1x04_Pitch2.54mm
- J4: value Analog_signal_female -> Analog_signal_male
- J6: value Servo_Power -> Servo_ground
- J7: value Encoder_Power -> encoder_power; footprint Pin_Headers:Pin_Header_Straight_1x06_Pitch2.54mm -> Pin_Headers:Pin_Header_Straight_1x04_Pitch2.54mm
- J8: value Analog_Power_female -> encoder_ground; footprint Pin_Headers:Pin_Header_Straight_1x08_Pitch2.54mm -> Pin_Headers:Pin_Header_Straight_1x04_Pitch2.54mm
- moved J4 83.8 mm to (200.7, 116.2), turned to 270 degrees
- moved J8 59.2 mm to (188.6, 80.0), turned to 90 degrees
- moved J2 36.2 mm to (196.2, 74.9), turned to 270 degrees
- moved J1 34.3 mm to (161.3, 116.2), turned to 90 degrees
- moved R2 32.2 mm to (168.4, 67.3)
- moved D9 31.6 mm to (162.6, 67.3), turned to 180 degrees
- moved J7 28.6 mm to (188.6, 77.5)
- moved R1 8.09 mm to (179.8, 67.3)
- moved D8 6.82 mm to (174.7, 67.3), turned to 180 degrees
- moved J6 2.54 mm to (138.4, 81.3)
Connections:
- J18 pad 3: /Encoder_6 -> Net-(J18-Pad3)
- J18 pad 4: /Encoder_5 -> Net-(J18-Pad4)
- J18 pad 5: /Encoder_4 -> Net-(J18-Pad5)
- J18 pad 6: /Encoder_3 -> Net-(J18-Pad6)
- J18 pad 7: /Encoder_2 -> Net-(J18-Pad7)
- J18 pad 8: /Encoder_1 -> Net-(J18-Pad8)
- J22 pad 1: /SDA -> /Encoder_1
- J22 pad 2: /SCL -> /Encoder_2
- J22 pad 3: Net-(J22-Pad3) -> /Encoder_3
- J22 pad 4: Net-(J22-Pad4) -> /Encoder_4
- J6 pad 1: +5V -> GND
- J6 pad 2: +5V -> GND
- J6 pad 3: +5V -> GND
- J6 pad 4: +5V -> GND
- J6 pad 5: +5V -> GND
- J6 pad 6: +5V -> GND
- J7 pad 3: +5V -> Net-(J7-Pad3)
- J8 pad 1: +5V -> GND
- J8 pad 2: +5V -> GND
- J8 pad 3: Net-(J8-Pad3) -> GND
- J8 pad 4: +5V -> GND
Routing:
- net +12V: track 75.3 -> 0.00 mm
- net /Drain_2: track 60.3 -> 0.00 mm
- net /Drain_3: track 36.6 -> 0.00 mm
- net /Drain_6: track 35.9 -> 0.00 mm
- net /Drain_5: track 29.5 -> 0.00 mm
- net /Drain_4: track 25.0 -> 0.00 mm
- net /Drain_1: track 11.8 -> 0.00 mm
- net /TX: track 0.00 -> 8.91 mm
- net /Servo_6: track 0.00 -> 5.45 mm
- net /Servo_5: track 0.00 -> 5.45 mm
- net /Servo_3: track 0.00 -> 5.45 mm
- net /Servo_2: track 0.00 -> 5.45 mm
- net /Servo_4: track 0.00 -> 5.45 mm
- net /Servo_1: track 0.00 -> 5.45 mm
- net /RX: track 0.00 -> 4.54 mm
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- added copper zone on F.Cu, net +5V
- added copper zone on F.Cu, net Net-(D1-Pad2)
- added copper zone on F.Cu, net Net-(F1-Pad1)
Other:
- board text added: "Noah Lohman Phoenixbot Arduino Shield 2018"
