File: _saved_Phoenix_Bot_arduino_shield.sch (KiCad schematic (older format))
At the start: 46 parts, among them J1 Analog_signal_male, J10 Ground, J11 Ground, J12 Ground, J13 12V_terminal, J14 PWN(10-5), J15 On Board Supply, J16 1x8 Male, J17 1x8 Male, J18 PWM_(6-1), J19 Analog_Pin_1, J2 Encoder_signal, J20 1x8 Female, J21 1x8 Female, J22 Serial, J23 ICSP, J24 Analog_Pin_2, J25 Digital_Pins, J27 Solenoid_terminal, J28 Solendoid_middle_terminal, J29 bottom_solenoid_terminal, J3 Servo_signal, J4 Analog_signal_female, J5 Analog_signal_power, J6 Servo_Power, J7 Encoder_Power, J8 Analog_Power_female, J9 Ground, q1 solenoid_1, q2 solenoid_4, q3 solenoid_3, q4 solenoid_5, q5 solenoid_3, q6 solenoid_6

Commit message: More progress on Board, mapped except solenoids
Parts:
- removed J10, J11: Ground, Pin_Headers:Pin_Header_Straight_1x06_Pitch2.54mm, symbol Conn_01x06_Male
- removed J12: Ground, Pin_Headers:Pin_Header_Straight_1x08_Pitch2.54mm, symbol Conn_01x08_Female
- removed J2: Encoder_signal, Pin_Headers:Pin_Header_Straight_1x06_Pitch2.54mm, symbol Conn_01x06_Male
- removed J5: Analog_signal_power, Pin_Headers:Pin_Header_Straight_1x08_Pitch2.54mm, symbol Conn_01x08_Male
- removed J7: Encoder_Power, Pin_Headers:Pin_Header_Straight_1x06_Pitch2.54mm, symbol Conn_01x06_Male
- removed J8: Analog_Power_female, Pin_Headers:Pin_Header_Straight_1x08_Pitch2.54mm, symbol Conn_01x08_Female
- removed J9: Ground, Pin_Headers:Pin_Header_Straight_1x08_Pitch2.54mm, symbol Conn_01x08_Male
- added J2: Encoder_Signal, Pin_Headers:Pin_Header_Straight_1x04_Pitch2.54mm, symbol Conn_01x04_Male
- added J7: encoder_power, Pin_Headers:Pin_Header_Straight_1x04_Pitch2.54mm, symbol Conn_01x04_Male
- added J8: encoder_ground, Pin_Headers:Pin_Header_Straight_1x04_Pitch2.54mm, symbol Conn_01x04_Male
- J4: value Analog_signal_female -> Analog_signal_male
- J6: value Servo_Power -> Servo_ground
Connections:
- net +5V: now also J7.1 (Pin_1), J7.2 (Pin_2), J7.4 (Pin_4); no longer J6.1 (Pin_1), J6.2 (Pin_2), J6.3 (Pin_3), J6.4 (Pin_4), J6.5 (Pin_5), J6.6 (Pin_6)
- net Encoder_1: now also J22.1 (Pin_1), J2.1 (Pin_1); no longer J18.8 (Pin_8)
- net Encoder_2: now also J22.2 (Pin_2), J2.2 (Pin_2); no longer J18.7 (Pin_7)
- net Encoder_3: now also J22.3 (Pin_3), J2.3 (Pin_3); no longer J18.6 (Pin_6)
- net Encoder_4: now also J22.4 (Pin_4), J2.4 (Pin_4); no longer J18.5 (Pin_5)
- net GND: now also J6.1 (Pin_1), J6.2 (Pin_2), J6.3 (Pin_3), J6.4 (Pin_4), J6.5 (Pin_5), J6.6 (Pin_6), J8.1 (Pin_1), J8.2 (Pin_2), J8.3 (Pin_3), J8.4 (Pin_4)
- net SCL: no longer J22.2 (Pin_2)
- net SDA: no longer J22.1 (Pin_1)
- net Encoder_5: no longer names the net of J18.4 (Pin_4)
- net Encoder_6: no longer names the net of J18.3 (Pin_3)
